File: kiCad/capm/capm.kicad_pcb (KiCad board)
At the start: 2 copper layers, 55 x 50 mm, 18 parts, among them J1 Conn_01x01_Female, J2 Conn_01x01_Female, J3 Conn_01x01_Female, J4 Conn_01x02_Female, J5 Conn_01x02_Female, U1 MCP6002-xSN, U2 MCP6542-xSN

Commit message: pcb update
Parts:
- removed the C2 at (135.0, 55.0)
- removed the C3 at (151.0, 80.0)
- removed C5, C6, C8: 100n, Capacitor_SMD:C_0805_2012Metric_Pad1.18x1.45mm_HandSolder
- removed the J5 at (130.5, 62.3)
- added J4: Conn_01x01_Female, Connector_PinHeader_2.54mm:PinHeader_1x01_P2.54mm_Vertical, F.Cu at (130.5, 62.5)
- added R1: 10k, Resistor_SMD:R_0805_2012Metric_Pad1.20x1.40mm_HandSolder, B.Cu at (142.0, 77.0)
- added R2: 10k, Resistor_SMD:R_0805_2012Metric_Pad1.20x1.40mm_HandSolder, B.Cu at (146.5, 77.0)
- U1, U2: footprint Package_DIP:DIP-8_W7.62mm_SMDSocket_SmallPads -> Package_SO:SO-8_3.9x4.9mm_P1.27mm
- moved J5 11.0 mm to (130.5, 67.0)
- moved R5 4.68 mm to (155.0, 56.5)
- moved R3 4.27 mm to (156.5, 60.0)
- moved R4 4.27 mm to (154.0, 60.0)
- moved C3 3.35 mm to (146.5, 52.0)
- moved C2 3.16 mm to (146.0, 69.0)
- renumbered C4 to C2, C7 to C3, J4 to J3, J3 to J5, R1 to R3, R2 to R4, R3 to R5
Connections:
- J3 pad 1: Net-(J4-Pad1) (its old number) -> Net-(J3-Pad1)
- J5 pad 1: -5V -> GND
- R3 pad 2: Net-(J4-Pad1) (its old number) -> Net-(J3-Pad1)
- U1 pad 2: GND -> Net-(J3-Pad1)
- U1 pad 3: Net-(J4-Pad1) (its old number) -> +3V0
- U1 pad 4: -5V -> GND
- U1 pad 5: GND -> Net-(R1-Pad1)
- U1 pad 6: GND -> +3V0
- U1 pad 7: unconnected-(U1-Pad7) -> +3V0
- U2 pad 2: GND -> +3V0
- U2 pad 4: -5V -> GND
Routing:
- net -5V: track 98.7 -> 0.00 mm, vias 4 -> 0
- net Net-(J3-Pad1): track 0.00 -> 47.7 mm, vias 0 -> 2
- net +3V0: track 0.00 -> 39.6 mm, vias 0 -> 2
- net Net-(J4-Pad1) (its old number): track 38.2 -> 0.00 mm, vias 2 -> 0
- net Net-(J4-Pad1): track 43.6 -> 38.3 mm
- net Net-(R1-Pad1): track 0.00 -> 4.13 mm
- net Net-(R4-Pad2): track 8.83 -> 5.98 mm
- net +5V: track 114.3 -> 115.3 mm, vias 0 -> 2
- net Net-(J3-Pad2): track 36.7 -> 37.3 mm
