File: kiCad/capm/capm.kicad_sch (KiCad schematic)
At the start: 18 parts, among them J1 Conn_01x01_Female, J2 Conn_01x01_Female, J3 Conn_01x01_Female, J4 Conn_01x02_Female, J5 Conn_01x02_Female, U1 MCP6002-xSN, U2 MCP6542-xSN

Commit message: pcb update
Parts:
- removed C2, C3, C5, C6, C8: 100n, Capacitor_SMD:C_0805_2012Metric_Pad1.18x1.45mm_HandSolder, symbol Device:C
- removed J5: Conn_01x02_Female, Connector_PinHeader_2.54mm:PinHeader_1x02_P2.54mm_Vertical, symbol Connector:Conn_01x02_Female
- added J4: Conn_01x01_Female, Connector_PinHeader_2.54mm:PinHeader_1x01_P2.54mm_Vertical, symbol Connector:Conn_01x01_Female
- added R1, R2: 10k, Resistor_SMD:R_0805_2012Metric_Pad1.20x1.40mm_HandSolder, symbol Device:R
- U1, U2: footprint Package_DIP:DIP-8_W7.62mm_SMDSocket_SmallPads -> Package_SO:SO-8_3.9x4.9mm_P1.27mm
- renumbered C4 to C2, C7 to C3, J4 to J3, J3 to J5, R1 to R3, R2 to R4, R3 to R5
Connections:
- net -5V is gone; now on net GND: J5.1 (Pin_1), U1.4 (V-), U2.4 (V-)
- net +5V: now also R1.2
- net GND: now also R2.1; no longer U1.2 (-), U1.5 (+), U1.6 (-), U2.2 (-)
- net at R3.1, R5.2, U2.1: now also J4.1 (Pin_1)
- net +3V0: now reaches U1.7
- net +3V0: now also U1.3 (+), U1.6 (-), U2.2 (-)
- net at J3.1 (Pin_1), R3.2: now also U1.2 (-); no longer U1.3 (+)
- new net: R1.1, R2.2, U1.5 (+)
Other:
- moved on the sheet: C2, C3, J5, U1B, U2B
